File: Base/Eagle/TurretController.brd (EAGLE design)
At the start: 123.2 x 100 mm, 88 parts, among them CN1 2EDG-2, IC1 LM2596S-5, IC2 MCP23017SO, Q1 BC818-16SMD, Q2 BC818-16SMD, Q3 BC818-16SMD, Q4 BC818-16SMD

Commit message: First corrections to board, addition of protection diodes
Parts:
- added D10, D11, D12, D9: SK34, Diodes:DO214AC
Connections:
- net N$10 renamed STEP
- net N$8 renamed DIR
- net GND: now also D10.A, D11.A, D12.A, D9.A, OK4.4
- net N$11: now also D9.C
- net N$3: now also D12.C
- net N$4: now also D11.C
- net N$9: now also D10.C
Routing:
- net N$9: track 14.1 -> 21.1 mm
- net N$11: track 14.1 -> 21.1 mm
- net N$4: track 14.5 -> 21.4 mm
- net N$3: track 14.1 -> 21.0 mm
Other:
- board text added: "DIR-/+"
- board text added: "STEP-/+"
- board text added: "Version 1.1"
- board text removed: "DIR+/-"
- board text removed: "STEP+/-"
- board text removed: "Version 1.0"
Changed lines of the file:
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@@
 <text x="97.663" y="97.409" size="1.778" layer="21">INDEX</text>
 <text x="121.285" y="50.546" size="1.778" layer="21" rot="R90">ANGULAR POSITION ENCODER</text>
-<text x="34.417" y="97.663" size="1.778" layer="21">STEP+/-</text>
-<text x="45.72" y="97.663" size="1.778" layer="21">DIR+/-</text>
+<text x="35.687" y="97.663" size="1.778" layer="21">DIR-/+</text>
+<text x="44.45" y="97.663" size="1.778" layer="21">STEP-/+</text>
 <text x="121.412" y="25.273" size="1.778" layer="21" rot="R90">LinuxCNC</text>
 <text x="80.899" y="2.159" size="1.778" layer="21">JOG+</text>
@@
 <text x="65.786" y="38.989" size="5.08" layer="21" font="vector">depronman</text>
 <text x="65.786" y="33.909" size="2.54" layer="21" font="vector">Turret Controller</text>
-<text x="65.786" y="28.829" size="2.54" layer="21" font="vector">Version 1.0</text>
+<text x="65.786" y="28.829" size="2.54" layer="21" font="vector">Version 1.1</text>
 <text x="66.04" y="39.116" size="5.08" layer="21" font="vector">depronman</text>
 </plain>
@@
 </element>
 <element name="D2" library="Diodes" package="SOD523" value="BAS516" x="17.78" y="64.77" smashed="yes" rot="R90">
-<attribute name="NAME" x="17.145" y="64.135" size="1.27" layer="25" rot="R90"/>
 <attribute name="VALUE" x="19.685" y="64.135" size="1.27" layer="27" rot="R90"/>
 </element>
 <element name="D3" library="Diodes" package="SOD523" value="BAS516" x="17.399" y="81.153" smashed="yes" rot="R90">
-<attribute name="NAME" x="16.764" y="80.518" size="1.27" layer="25" rot="R90"/>
 <attribute name="VALUE" x="19.304" y="80.518" size="1.27" layer="27" rot="R90"/>
 </element>
 <element name="D4" library="Diodes" package="SOD523" value="BAS516" x="17.78" y="48.26" smashed="yes" rot="R90">
-<attribute name="NAME" x="17.145" y="47.625" size="1.27" layer="25" rot="R90"/>
 <attribute name="VALUE" x="19.685" y="47.625" size="1.27" layer="27" rot="R90"/>
 </element>
 <element name="D6" library="Diodes" package="SOD523" value="BAS516" x="17.78" y="31.75" smashed="yes" rot="R90">
-<attribute name="NAME" x="17.145" y="31.115" size="1.27" layer="25" rot="R90"/>
 <attribute name="VALUE" x="19.685" y="31.115" size="1.27" layer="27" rot="R90"/>
 </element>
@@
 <attribute name="SPICEPREFIX" value="R" x="106.68" y="41.91" size="1.778" layer="27" display="off"/>
 <attribute name="VALUE" x="106.045" y="39.37" size="1.27" layer="27"/>
+</element>
+<element name="D9" library="Diodes" package="DO214AC" value="SK34" x="14.605" y="81.153" smashed="yes" rot="R270">
+<attribute name="SPICEPREFIX" value="D" x="14.605" y="81.153" size="1.778" layer="27" rot="R270" display="off"/>
+</element>
+<element name="D10" library="Diodes" package="DO214AC" value="SK34" x="14.605" y="64.643" smashed="yes" rot="R270">
+<attribute name="SPICEPREFIX" value="D" x="14.605" y="64.643" size="1.778" layer="27" rot="R270" display="off"/>
+</element>
+<element name="D11" library="Diodes" package="DO214AC" value="SK34" x="14.478" y="48.133" smashed="yes" rot="R270">
+<attribute name="SPICEPREFIX" value="D" x="14.478" y="48.133" size="1.778" layer="27" rot="R270" display="off"/>
+</element>
+<element name="D12" library="Diodes" package="DO214AC" value="SK34" x="14.478" y="31.623" smashed="yes" rot="R270">
+<attribute name="SPICEPREFIX" value="D" x="14.478" y="31.623" size="1.778" layer="27" rot="R270" display="off"/>
 </element>
 </elements>
@@
 <wire x1="7.62" y1="33.655" x2="19.05" y2="33.655" width="1.27" layer="16"/>
 <wire x1="19.05" y1="33.655" x2="20.955" y2="31.75" width="1.27" layer="16"/>
+<contactref element="D12" pad="C"/>
+<wire x1="7.62" y1="33.655" x2="14.46" y2="33.655" width="0.8128" layer="1"/>
+<wire x1="14.46" y1="33.655" x2="14.478" y2="33.673" width="0.8128" layer="1"/>
 </signal>
 <signal name="N$4">
@@
 <wire x1="19.685" y1="50.165" x2="20.955" y2="48.895" width="1.27" layer="16"/>
 <wire x1="20.955" y1="48.895" x2="20.955" y2="48.26" width="1.27" layer="16"/>
+<contactref element="D11" pad="C"/>
+<wire x1="7.62" y1="50.165" x2="14.46" y2="50.165" width="0.8128" layer="1"/>
+<wire x1="14.46" y1="50.165" x2="14.478" y2="50.183" width="0.8128" layer="1"/>
 </signal>
 <signal name="N$9">
@@
 <wire x1="7.62" y1="66.675" x2="19.05" y2="66.675" width="1.27" layer="16"/>
 <wire x1="19.05" y1="66.675" x2="20.955" y2="64.77" width="1.27" layer="16"/>
+<contactref element="D10" pad="C"/>
+<wire x1="7.62" y1="66.675" x2="14.587" y2="66.675" width="0.8128" layer="1"/>
+<wire x1="14.587" y1="66.675" x2="14.605" y2="66.693" width="0.8128" layer="1"/>
 </signal>
 <signal name="N$11">
@@
 <wire x1="7.62" y1="83.185" x2="19.05" y2="83.185" width="1.27" layer="16"/>
 <wire x1="19.05" y1="83.185" x2="20.955" y2="81.28" width="1.27" layer="16"/>
+<contactref element="D9" pad="C"/>
+<wire x1="7.62" y1="83.185" x2="14.587" y2="83.185" width="0.8128" layer="1"/>
+<wire x1="14.587" y1="83.185" x2="14.605" y2="83.203" width="0.8128" layer="1"/>
 </signal>
 <signal name="GND">
@@
 <wire x1="86.06" y1="67.31" x2="86.06" y2="66.04" width="0.254" layer="1"/>
 <wire x1="86.06" y1="66.04" x2="86.06" y2="64.77" width="0.254" layer="1"/>
+<contactref element="OK4" pad="4"/>
+<contactref element="D12" pad="A"/>
+<contactref element="D11" pad="A"/>
+<contactref element="D10" pad="A"/>
+<contactref element="D9" pad="A"/>
 </signal>
 <signal name="N$19" class="1">
@@
 <wire x1="84.709" y1="88.011" x2="93.919" y2="88.011" width="0.3048" layer="1"/>
 </signal>
-<signal name="N$8">
+<signal name="DIR">
 <contactref element="U$1" pad="D12"/>
 <contactref element="J6" pad="3"/>
@@
 <wire x1="69.85" y1="88.392" x2="66.548" y2="91.694" width="0.3048" layer="1"/>
 </signal>
-<signal name="N$10">
+<signal name="STEP">
 <contactref element="J6" pad="1"/>
 <contactref element="U$1" pad="D11"/>
